Commit message: V-Final

File: Marco Izeppi/ROS/Espacios de simulacion/simulation_ws/src/two_wheel_description/urdf/two_wheel.xacro (robot description, xacro)
@@ -1,9 +1,8 @@
 <?xml version="1.0" ?>
 <robot name="two_wheel" xmlns:xacro="https://www.ros.org/wiki/xacro" >
-  <!-- include the xacro files-->
   <xacro:include filename="$(find two_wheel_description)/urdf/materials.xacro" />
   <xacro:include filename="$(find two_wheel_description)/urdf/two_wheel.gazebo" />
   <xacro:include filename="$(find two_wheel_description)/urdf/macro.xacro" />
-  <!-- Chasis defined here -->
+  <!-- definicion de dimensiones del robot -->
   <link name="link_chassis">
     <pose>0 0 0.1 0 0 0</pose>
@@ -15,5 +14,5 @@
     <collision name="collision_chassis">
       <geometry>
-        <box size="0.5 0.3 0.07"/>
+        <cylinder radius="0.17" length="0.1"/>
       </geometry>
     </collision>
@@ -21,11 +20,10 @@
       <origin rpy="0 0 0" xyz="0 0 0"/>
       <geometry>
-        <box size="0.5 0.3 0.07"/>
+        <cylinder radius="0.17" length="0.1"/>
       </geometry>
       <material name="blue"/>
     </visual>
-    <!-- caster front -->
     <collision name="caster_front_collision">
-      <origin rpy=" 0 0 0" xyz="0.35 0 -0.05"/>
+      <origin rpy=" 0 0 0" xyz="0.1 0 -0.05"/>
       <geometry>
         <sphere radius="0.05"/>
@@ -43,5 +41,5 @@
     </collision>
     <visual name="caster_front_visual">
-      <origin rpy=" 0 0 0" xyz="0.2 0 -0.05"/>
+      <origin rpy=" 0 0 0" xyz="0.1 0 -0.05"/>
       <geometry>
         <sphere radius="0.05"/>
@@ -49,8 +47,8 @@
     </visual>
     </link>
-  <!-- Create wheel right -->
+  <!-- creacion de la rueda derecha -->
    <xacro:link_wheel name="link_right_wheel" />
    <xacro:joint_wheel name="joint_right_wheel"  child="link_right_wheel"  origin_xyz="-0.05 0.15 0"  />
-  <!-- Left Wheel link -->
+  <!-- creacion de la rueda izquierda -->
   <xacro:link_wheel name="link_left_wheel" />
   <xacro:joint_wheel name="joint_left_wheel"   child="link_left_wheel"   origin_xyz="-0.05 -0.15 0"  />
@@ -59,11 +57,10 @@
       <origin xyz="0 0 0" rpy="0 0 0" />
       <mass value="1" />
-      <!-- RANDOM INERTIA BELOW -->
-      <xacro:cylinder_inertia mass="1" r="0.05" l="0.1" />>
+      <xacro:cylinder_inertia mass="1" r="0.05" l="0.05" />>
     </inertial>
     <visual>
       <origin xyz="0 0 0" rpy="0 0 0" />
       <geometry>
-        <cylinder radius="0.05" length="0.1"/>
+        <cylinder radius="0.05" length="0.05"/>
       </geometry>
       <material name="white" />
@@ -77,5 +74,5 @@
   </link>
   <joint name="joint_sensor_laser" type="fixed">
-    <origin xyz="0.15 0 0.05" rpy="0 0 0"/>
+    <origin xyz="0 0 0.05" rpy="0 0 0"/>
     <parent link="link_chassis"/>
     <child link="sensor_laser"/>
